Commit message: update about robotiq_2f85 gripper

File: Asset/Robot/mobile_manipulator/arm/flexiv/urdf/flexiv_rizon4_robotiq_2f85.urdf (robot description, URDF)
Before this commit: robot rizon4, 17 links, 16 joints
Links:
- removed link robotiq_85_base_link
- added link left_inner_finger_pad, mass 1.; collision box size=0.022 0.00635 0.0375; visual box size=0.022 0.00635 0.0375
- added link right_inner_finger_pad, mass 1; collision box size=0.022 0.00635 0.0375; visual box size=0.022 0.00635 0.0375
- added link robotiq_arg2f_base_link, mass 0.22652; collision mesh filename=../../../end_effector/gripper/robotiq_85/collision/robotiq_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; visual mesh filename=../../../end_effector/gripper/robotiq_85/visual/robotiq_arg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 scale=0.001 0.001 0.001
- link left_inner_finger: mass 0.00724255346165745 -> 0.0104003125914103; geometry collision mesh filename=../../../end_effector/gripper/robotiq_85/collision/robotiq_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 scale=0.001 0.001 0.001; visual mesh filename=../../../end_effector/gripper/robotiq_85/visual/robotiq_arg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 scale=0.001 0.001 0.001
- link left_inner_knuckle: mass 0.0110930853895903 -> 0.0271177346495152; geometry collision mesh filename=../../../end_effector/gripper/robotiq_85/collision/robotiq_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 scale=0.001 0.001 0.001; visual mesh filename=../../../end_effector/gripper/robotiq_85/visual/robotiq_arg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 scale=0.001 0.001 0.001
- link left_outer_finger: mass 0.0273093985570947 -> 0.022614240507152; geometry collision mesh filename=../../../end_effector/gripper/robotiq_85/collision/robotiq_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 scale=0.001 0.001 0.001; visual mesh filename=../../../end_effector/gripper/robotiq_85/visual/robotiq_arg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 scale=0.001 0.001 0.001
- link left_outer_knuckle: mass 0.00684838849434396 -> 0.00853198276973456; geometry collision mesh filename=../../../end_effector/gripper/robotiq_85/collision/robotiq_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 scale=0.001 0.001 0.001; visual mesh filename=../../../end_effector/gripper/robotiq_85/visual/robotiq_arg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 scale=0.001 0.001 0.001
- link right_inner_finger: mass 0.00724255346165744 -> 0.0104003125914103; geometry collision mesh filename=../../../end_effector/gripper/robotiq_85/collision/robotiq_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 scale=0.001 0.001 0.001; visual mesh filename=../../../end_effector/gripper/robotiq_85/visual/robotiq_arg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 scale=0.001 0.001 0.001
- link right_inner_knuckle: mass 0.0110930853895903 -> 0.0271177346495152; geometry collision mesh filename=../../../end_effector/gripper/robotiq_85/collision/robotiq_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 scale=0.001 0.001 0.001; visual mesh filename=../../../end_effector/gripper/robotiq_85/visual/robotiq_arg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 scale=0.001 0.001 0.001
- link right_outer_finger: mass 0.0273093985570947 -> 0.022614240507152; geometry collision mesh filename=../../../end_effector/gripper/robotiq_85/collision/robotiq_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 scale=0.001 0.001 0.001; visual mesh filename=../../../end_effector/gripper/robotiq_85/visual/robotiq_arg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 scale=0.001 0.001 0.001
- link right_outer_knuckle: mass 0.00684838849401352 -> 0.00853198276973456; geometry collision mesh filename=../../../end_effector/gripper/robotiq_85/collision/robotiq_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 scale=0.001 0.001 0.001; visual mesh filename=../../../end_effector/gripper/robotiq_85/visual/robotiq_arg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 scale=0.001 0.001 0.001
Joints:
- added joint left_inner_finger_pad_joint: type fixed, parent left_inner_finger, child left_inner_finger_pad, origin xyz=0 -0.0220203446692936 0.03242 rpy=0 0 0, axis 0 0 1
- added joint right_inner_finger_pad_joint: type fixed, parent right_inner_finger, child right_inner_finger_pad, origin xyz=0 -0.0220203446692936 0.03242 rpy=0 0 0, axis 0 0 1
- joint arm_connect_gripper: child robotiq_85_base_link -> robotiq_arg2f_base_link
- joint finger_joint: axis 0 -1 0 -> 1 0 0; limit lower=0 upper=0.725 effort=1000 velocity=2.0 -> lower=0 upper=0.8 effort=1000 velocity=2.0; origin xyz=0.0306011444260539 0 0.0627920162695395 rpy=0 0 0 -> xyz=0 -0.0306011 0.054904 rpy=0 0 3.14159265359; parent robotiq_85_base_link -> robotiq_arg2f_base_link
- joint left_inner_finger_joint: axis 0 -1 0 -> 1 0 0; limit lower=0 upper=0.8757 effort=1000 velocity=2.0 -> lower=-0.8757 upper=0 effort=1000 velocity=2.0; origin xyz=0.034585310861294 0 0.0454970193817975 rpy=0 0 0 -> xyz=0 0.0061 0.0471 rpy=0 0 0; parent left_inner_knuckle -> left_outer_finger
- joint left_inner_knuckle_joint: axis 0 -1 0 -> 1 0 0; origin xyz=0.0127000000001501 0 0.0693074999999639 rpy=0 0 0 -> xyz=0 -0.0127 0.06142 rpy=0 0 3.14159265359; parent robotiq_85_base_link -> robotiq_arg2f_base_link
- joint left_outer_finger_joint: axis 0 -1 0 -> 1 0 0; origin xyz=0.0316910442266543 0 -0.00193396375724605 rpy=0 0 0 -> xyz=0 0.0315 -0.0041 rpy=0 0 0
- joint right_inner_finger_joint: axis 0 1 0 -> 1 0 0; limit lower=0 upper=0.8757 effort=1000 velocity=2.0 -> lower=-0.8757 upper=0 effort=1000 velocity=2.0; mimic joint=finger_joint multiplier=1 offset=0 -> joint=finger_joint multiplier=-1 offset=0; origin xyz=0.0341060475457406 0 0.0458573878541688 rpy=0 0 0 -> xyz=0 0.0061 0.0471 rpy=0 0 0; parent right_inner_knuckle -> right_outer_finger
- joint right_inner_knuckle_joint: axis 0 1 0 -> 1 0 0; mimic joint=finger_joint multiplier=-1 offset=0 -> joint=finger_joint multiplier=1 offset=0; origin xyz=-0.0126999999998499 0 0.0693075000000361 rpy=0 0 3.14159265358979 -> xyz=0 0.0127 0.06142 rpy=0 0 0.0; parent robotiq_85_base_link -> robotiq_arg2f_base_link
- joint right_outer_finger_joint: axis 0 1 0 -> 1 0 0; origin xyz=0.0317095909367246 0 -0.0016013564954687 rpy=0 0 0 -> xyz=0 0.0315 -0.0041 rpy=0 0 0
- joint right_outer_knuckle_joint: axis 0 1 0 -> 1 0 0; limit lower=0 upper=0.8757 effort=1000 velocity=2.0 -> lower=0 upper=0.81 effort=1000 velocity=2.0; mimic joint=finger_joint multiplier=-1 offset=0 -> joint=finger_joint multiplier=1 offset=0; origin xyz=-0.0306011444258893 0 0.0627920162695395 rpy=0 0 3.14159265358979 -> xyz=0 0.0306011 0.054904 rpy=0 0 0; parent robotiq_85_base_link -> robotiq_arg2f_base_link

Commit message: integrate robotiq 2f85 control from pybullet ur5e robotiq codebase

File: Asset/Robot/mobile_manipulator/arm/flexiv/urdf/flexiv_rizon4_robotiq_2f85.urdf (robot description, URDF)
Before this commit: robot rizon4, 19 links, 18 joints
Links:
- added link ee_link; collision box size=0.01 0.01 0.01
- link left_inner_finger: geometry collision mesh filename=../../../end_effector/gripper/robotiq_2f85/meshes/v2/collis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 scale=0.001 0.001 0.001; visual mesh filename=../../../end_effector/gripper/robotiq_2f85/meshes/v2/visual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 scale=0.001 0.001 0.001
- link left_inner_knuckle: geometry collision mesh filename=../../../end_effector/gripper/robotiq_2f85/meshes/v2/collis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 scale=0.001 0.001 0.001; visual mesh filename=../../../end_effector/gripper/robotiq_2f85/meshes/v2/visual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 scale=0.001 0.001 0.001
- link left_outer_finger: geometry collision mesh filename=../../../end_effector/gripper/robotiq_2f85/meshes/v2/collis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 scale=0.001 0.001 0.001; visual mesh filename=../../../end_effector/gripper/robotiq_2f85/meshes/v2/visual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 scale=0.001 0.001 0.001
- link left_outer_knuckle: geometry collision mesh filename=../../../end_effector/gripper/robotiq_2f85/meshes/v2/collis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 scale=0.001 0.001 0.001; visual mesh filename=../../../end_effector/gripper/robotiq_2f85/meshes/v2/visual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 scale=0.001 0.001 0.001
- link right_inner_finger: geometry collision mesh filename=../../../end_effector/gripper/robotiq_2f85/meshes/v2/collis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 scale=0.001 0.001 0.001; visual mesh filename=../../../end_effector/gripper/robotiq_2f85/meshes/v2/visual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 scale=0.001 0.001 0.001
- link right_inner_knuckle: geometry collision mesh filename=../../../end_effector/gripper/robotiq_2f85/meshes/v2/collis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 scale=0.001 0.001 0.001; visual mesh filename=../../../end_effector/gripper/robotiq_2f85/meshes/v2/visual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 scale=0.001 0.001 0.001
- link right_outer_finger: geometry collision mesh filename=../../../end_effector/gripper/robotiq_2f85/meshes/v2/collis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 scale=0.001 0.001 0.001; visual mesh filename=../../../end_effector/gripper/robotiq_2f85/meshes/v2/visual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 scale=0.001 0.001 0.001
- link right_outer_knuckle: geometry collision mesh filename=../../../end_effector/gripper/robotiq_2f85/meshes/v2/collis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 scale=0.001 0.001 0.001; visual mesh filename=../../../end_effector/gripper/robotiq_2f85/meshes/v2/visual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 scale=0.001 0.001 0.001
- link robotiq_arg2f_base_link: geometry collision mesh filename=../../../end_effector/gripper/robotiq_2f85/meshes/v2/collis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; visual mesh filename=../../../end_effector/gripper/robotiq_2f85/meshes/v2/visual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 scale=0.001 0.001 0.001
Joints:
- added joint ee_fixed_joint: type fixed, parent link7, child ee_link, origin xyz=0.0 0。0 0.0 rpy=0.0 0.0 1.57079632679
- joint arm_connect_gripper: parent link7 -> ee_link

File: Asset/Robot/mobile_manipulator/arm/universal/urdf/ur5e_vacuum_long.urdf (robot description, URDF)
Before this commit: robot ur5e_vacuum_long, 13 links, 12 joints
Links:
- link base_link: geometry collision mesh filename=../meshes/ur5e/v1/base.stl scale=1.00000 1.00000 1.00000; visual mesh filename=../meshes/ur5e/v1/base.stl scale=1.00000 1.00000 1.00000
- link forearm_link: geometry collision mesh filename=../meshes/ur5e/v1/forearm.stl scale=1.00000 1.00000 1.00000; visual mesh filename=../meshes/ur5e/v1/forearm.stl scale=1.00000 1.00000 1.00000
- link lite_vacuum_gripper_link: geometry visual mesh filename=../meshes/ur5e/v1/base.stl scale=0.00100 0.00100 0.00100
- link shoulder_link: geometry collision mesh filename=../meshes/ur5e/v1/shoulder.stl scale=1.00000 1.00000 1.00000; visual mesh filename=../meshes/ur5e/v1/shoulder.stl scale=1.00000 1.00000 1.00000
- link upper_arm_link: geometry collision mesh filename=../meshes/ur5e/v1/upperarm.stl scale=1.00000 1.00000 1.00000; visual mesh filename=../meshes/ur5e/v1/upperarm.stl scale=1.00000 1.00000 1.00000
- link wrist_1_link: geometry collision mesh filename=../meshes/ur5e/v1/wrist1.stl scale=1.00000 1.00000 1.00000; visual mesh filename=../meshes/ur5e/v1/wrist1.stl scale=1.00000 1.00000 1.00000
- link wrist_2_link: geometry collision mesh filename=../meshes/ur5e/v1/wrist2.stl scale=1.00000 1.00000 1.00000; visual mesh filename=../meshes/ur5e/v1/wrist2.stl scale=1.00000 1.00000 1.00000
- link wrist_3_link: geometry collision mesh filename=../meshes/ur5e/v1/wrist3.stl scale=1.00000 1.00000 1.00000; visual mesh filename=../meshes/ur5e/v1/wrist3.stl scale=1.00000 1.00000 1.00000
